Commit message: xboxコントローラで動かした

File: install/0525_arm_description/share/0525_arm_description/urdf/0525_arm.urdf (robot description, URDF)
Before this commit: robot 0525_arm, 10 links, 9 joints
Joints:
- removed joint Revolute 1
- removed joint Revolute 2
- removed joint Revolute 3
- removed joint Revolute 4
- removed joint Revolute 5
- removed joint Revolute 6
- removed joint Rigid 7
- removed joint Slider 1
- removed joint Slider 2
- added joint Revolute_1: type continuous, parent base_link, child link1_1, origin xyz=0.0 0.0 0.0555 rpy=0 0 0, axis -0.0 0.0 1.0
- added joint Revolute_2: type continuous, parent link1_1, child link2_1, origin xyz=-3.7e-05 0.024464 0.06805 rpy=0 0 0, axis -0.000898 1.0 -0.0
- added joint Revolute_3: type continuous, parent link2_1, child link3_1, origin xyz=0.034905 -0.060969 0.35175 rpy=0 0 0, axis 0.000898 -1.0 -0.0
- added joint Revolute_4: type continuous, parent link3_1, child link4_1, origin xyz=0.325567 0.036793 -0.0001 rpy=0 0 0, axis 1.0 0.000898 0.0
- added joint Revolute_5: type continuous, parent link4_1, child link5_1, origin xyz=0.078683 0.019071 0.0 rpy=0 1.57 0, axis -0.000898 1.0 0.0
- added joint Revolute_6: type continuous, parent link5_1, child link6_1, origin xyz=0.064817 -0.018842 0.0 rpy=0 0 0, axis 1.0 0.000898 0.0
- added joint Rigid_7: type fixed, parent link6_1, child EndEffector_1, origin xyz=0.045 4e-05 -5e-05 rpy=0 0 0
- added joint Slider_1: type prismatic, parent EndEffector_1, child right_finger_1, origin xyz=0.007999 3e-05 0.055 rpy=0 0 0, axis 0.0 0.0 -1.0, limit lower=0.0 upper=0.024 effort=100 velocity=100
- added joint Slider_2: type prismatic, parent EndEffector_1, child left_finger_1, origin xyz=0.008 -1.6e-05 -0.055 rpy=0 0 0, axis 0.0 0.0 -1.0, limit lower=-0.024 upper=0.0 effort=100 velocity=100, mimic joint=Slider_1 multiplier=-1.0 offset=0.0

File: install/robot_config/share/robot_config/config/0525_arm.ros2_control.xacro (robot description, xacro)
@@ -12,57 +12,65 @@
                 </xacro:unless>
             </hardware>
-            <joint name="Revolute 1">
+            <joint name="Revolute_1">
                 <command_interface name="position"/>
+                <command_interface name="velocity"/>
                 <state_interface name="position">
-                  <param name="initial_value">${initial_positions['Revolute 1']}</param>
+                  <param name="initial_value">${initial_positions['Revolute_1']}</param>
                 </state_interface>
                 <state_interface name="velocity"/>
             </joint>
-            <joint name="Revolute 2">
+            <joint name="Revolute_2">
                 <command_interface name="position"/>
+                <command_interface name="velocity"/>
                 <state_interface name="position">
-                  <param name="initial_value">${initial_positions['Revolute 2']}</param>
+                  <param name="initial_value">${initial_positions['Revolute_2']}</param>
                 </state_interface>
                 <state_interface name="velocity"/>
             </joint>
-            <joint name="Revolute 3">
+            <joint name="Revolute_3">
                 <command_interface name="position"/>
+                <command_interface name="velocity"/>
                 <state_interface name="position">
-                  <param name="initial_value">${initial_positions['Revolute 3']}</param>
+                  <param name="initial_value">${initial_positions['Revolute_3']}</param>
                 </state_interface>
                 <state_interface name="velocity"/>
             </joint>
-            <joint name="Revolute 4">
+            <joint name="Revolute_4">
                 <command_interface name="position"/>
+                <command_interface name="velocity"/>
                 <state_interface name="position">
-                  <param name="initial_value">${initial_positions['Revolute 4']}</param>
+                  <param name="initial_value">${initial_positions['Revolute_4']}</param>
                 </state_interface>
                 <state_interface name="velocity"/>
             </joint>
-            <joint name="Revolute 5">
+            <joint name="Revolute_5">
                 <command_interface name="position"/>
+                <command_interface name="velocity"/>
                 <state_interface name="position">
-                  <param name="initial_value">${initial_positions['Revolute 5']}</param>
+                  <param name="initial_value">${initial_positions['Revolute_5']}</param>
                 </state_interface>
                 <state_interface name="velocity"/>
             </joint>
-            <joint name="Revolute 6">
+            <joint name="Revolute_6">
                 <command_interface name="position"/>
+                <command_interface name="velocity"/>
                 <state_interface name="position">
-                  <param name="initial_value">${initial_positions['Revolute 6']}</param>
+                  <param name="initial_value">${initial_positions['Revolute_6']}</param>
                 </state_interface>
                 <state_interface name="velocity"/>
             </joint>
-            <joint name="Slider 1">
+            <joint name="Slider_1">
                 <command_interface name="position"/>
+                <command_interface name="velocity"/>
                 <state_interface name="position">
-                  <param name="initial_value">${initial_positions['Slider 1']}</param>
+                  <param name="initial_value">${initial_positions['Slider_1']}</param>
                 </state_interface>
                 <state_interface name="velocity"/>
             </joint>
-            <joint name="Slider 2">
+            <joint name="Slider_2">
                 <command_interface name="position"/>
+                <command_interface name="velocity"/>
                 <state_interface name="position">
-                  <param name="initial_value">${initial_positions['Slider 2']}</param>
+                  <param name="initial_value">${initial_positions['Slider_2']}</param>
                 </state_interface>
                 <state_interface name="velocity"/>

File: install/robot_config/share/robot_config/config/0525_arm.urdf.xacro (robot description, xacro)
@@ -18,11 +18,11 @@
         </transmission>
     </xacro:macro>
-    <xacro:transmission_block joint_name="Revolute 1"/>
-    <xacro:transmission_block joint_name="Revolute 2"/>
-    <xacro:transmission_block joint_name="Revolute 3"/>
-    <xacro:transmission_block joint_name="Revolute 4"/>
-    <xacro:transmission_block joint_name="Revolute 5"/>
-    <xacro:transmission_block joint_name="Revolute 6"/>
-    <xacro:transmission_block joint_name="Slider 1"/>
-    <xacro:transmission_block joint_name="Slider 2"/>
+    <xacro:transmission_block joint_name="Revolute_1"/>
+    <xacro:transmission_block joint_name="Revolute_2"/>
+    <xacro:transmission_block joint_name="Revolute_3"/>
+    <xacro:transmission_block joint_name="Revolute_4"/>
+    <xacro:transmission_block joint_name="Revolute_5"/>
+    <xacro:transmission_block joint_name="Revolute_6"/>
+    <xacro:transmission_block joint_name="Slider_1"/>
+    <xacro:transmission_block joint_name="Slider_2"/>
 </robot>
