Commit message: フィールドとアーム一体のurdfを出力した

File: install/field_description/share/field_description/urdf/field.urdf (robot description, URDF)
Before this commit: robot field, 1 links, 0 joints
Links:
- link base_link: geometry collision mesh filename=file:///home/a/ws_moveit2/src/field_description-20250804T03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 scale=0.001 0.001 0.001; visual mesh filename=file:///home/a/ws_moveit2/src/field_description-20250804T03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 scale=0.001 0.001 0.001

File: src/field_description-20250804T033832Z-1-001/field_description/urdf/field.urdf (robot description, URDF)
Before this commit: robot field, 1 links, 0 joints
Links:
- link base_link: geometry collision mesh filename=file:///home/a/ws_moveit2/src/field_description-20250804T03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 scale=0.001 0.001 0.001; visual mesh filename=file:///home/a/ws_moveit2/src/field_description-20250804T03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 scale=0.001 0.001 0.001
