Commit message: unityにobject配置した

File: install/robot_config/share/robot_config/config/dual_arm.urdf.xacro (robot description, xacro)
@@ -230,9 +230,9 @@
         </joint>
         <joint name="${prefix}Revolute_3" type="revolute">
-            <origin rpy="0 0 0" xyz="0.034861 -0.011969 0.43175"/>
+            <origin rpy="0 -1.570796 0" xyz="0.034861 -0.011969 0.43175"/>
             <parent link="${prefix}link2_1"/>
             <child link="${prefix}link3_1"/>
             <axis xyz="-0.000898 1.0 0.0"/>
-            <limit effort="100" lower="-1.570796" upper="1.570796" velocity="100"/>
+            <limit effort="100" lower="-1.570796" upper="3.14159265359" velocity="100"/>
         </joint>
         <joint name="${prefix}Revolute_4" type="continuous">

File: src/urdf_0816_description-20250818T025130Z-1-001/urdf_0816_description/urdf/urdf_0816.urdf (robot description, URDF)
Before this commit: robot urdf_0816, 10 links, 9 joints
Joints:
- joint Revolute_3: origin xyz=0.034861 -0.011969 0.43175 rpy=0 0 0 -> xyz=0.034861 -0.011969 0.43175 rpy=0 -1.570796 0

Commit message: guiにALLREBOOTとALLTOLQUEON・OFFボタンを追加

File: install/robot_config/share/robot_config/config/dual_arm.urdf.xacro (robot description, xacro)
@@ -26,4 +26,6 @@
     <xacro:arg name="left_Revolute_3_lower_limit" default="-1.570796"/>
     <xacro:arg name="left_Revolute_3_upper_limit" default="3.14159265359"/>
+    <xacro:arg name="left_Revolute_6_lower_limit" default="-1.570796"/>
+    <xacro:arg name="left_Revolute_6_upper_limit" default="1.570796"/>
     <xacro:arg name="left_Slider_1_lower_limit" default="0.0"/>
     <xacro:arg name="left_Slider_1_upper_limit" default="0.024"/>
@@ -37,4 +39,6 @@
     <xacro:arg name="right_Revolute_3_lower_limit" default="-1.570796"/>
     <xacro:arg name="right_Revolute_3_upper_limit" default="3.14159265359"/>
+    <xacro:arg name="right_Revolute_6_lower_limit" default="-1.570796"/>
+    <xacro:arg name="right_Revolute_6_upper_limit" default="1.570796"/>
     <xacro:arg name="right_Slider_1_lower_limit" default="0.0"/>
     <xacro:arg name="right_Slider_1_upper_limit" default="0.024"/>
@@ -303,9 +307,10 @@
             <axis xyz="-0.000898 1.0 0.0"/>
         </joint>
-        <joint name="${prefix}Revolute_6" type="continuous">
+        <joint name="${prefix}Revolute_6" type="revolute">
             <origin rpy="${Revolute_6_rpy}" xyz="${Revolute_6_xyz}"/>
             <parent link="${prefix}link5_1"/>
             <child link="${prefix}link6_1"/>
             <axis xyz="0.0 0.0 -1.0"/>
+            <limit lower="$(arg ${prefix}Revolute_6_lower_limit)" upper="$(arg ${prefix}Revolute_6_upper_limit)" effort="300" velocity="10"/>
         </joint>
         <joint name="${prefix}Rigid_7" type="fixed">

Commit message: 無駄な回転を減らしてみれたかも

File: install/robot_config/share/robot_config/config/dual_arm.urdf.xacro (robot description, xacro)
@@ -26,4 +26,6 @@
     <xacro:arg name="left_Revolute_3_lower_limit" default="-1.570796"/>
     <xacro:arg name="left_Revolute_3_upper_limit" default="3.14159265359"/>
+    <xacro:arg name="left_Revolute_4_lower_limit" default="-1.570796"/>
+    <xacro:arg name="left_Revolute_4_upper_limit" default="1.570796"/>
     <xacro:arg name="left_Revolute_6_lower_limit" default="-1.570796"/>
     <xacro:arg name="left_Revolute_6_upper_limit" default="1.570796"/>
@@ -39,4 +41,6 @@
     <xacro:arg name="right_Revolute_3_lower_limit" default="-1.570796"/>
     <xacro:arg name="right_Revolute_3_upper_limit" default="3.14159265359"/>
+    <xacro:arg name="right_Revolute_4_lower_limit" default="-1.570796"/>
+    <xacro:arg name="right_Revolute_4_upper_limit" default="1.570796"/>
     <xacro:arg name="right_Revolute_6_lower_limit" default="-1.570796"/>
     <xacro:arg name="right_Revolute_6_upper_limit" default="1.570796"/>
@@ -295,9 +299,10 @@
             <limit effort="100" lower="$(arg ${prefix}Revolute_3_lower_limit)" upper="$(arg ${prefix}Revolute_3_upper_limit)" velocity="100"/>
         </joint>
-        <joint name="${prefix}Revolute_4" type="continuous">
+        <joint name="${prefix}Revolute_4" type="revolute">
             <origin rpy="${Revolute_4_rpy}" xyz="${Revolute_4_xyz}"/>
             <parent link="${prefix}link3_1"/>
             <child link="${prefix}link4_1"/>
             <axis xyz="1.0 0.000898 0.0"/>
+            <limit effort="100" lower="$(arg ${prefix}Revolute_4_lower_limit)" upper="$(arg ${prefix}Revolute_4_upper_limit)" velocity="100"/>
         </joint>
         <joint name="${prefix}Revolute_5" type="continuous">

Commit message: 整列機をslider jointで動かせるように

File: install/robot_config/share/robot_config/config/dual_arm.urdf.xacro (robot description, xacro)
@@ -516,3 +516,151 @@
         Slider_2_rpy="0 0 0"
     />
+    <!-- Materials for seiretu robots -->
+    <material name="blue_seiretu_steel_satin">
+        <color rgba="0.6274509803921569 0.6274509803921569 0.6274509803921569 1.0"/>
+    </material>
+    <material name="red_seiretu_steel_satin">
+        <color rgba="0.6274509803921569 0.6274509803921569 0.6274509803921569 1.0"/>
+    </material>
+    <!-- Blue Seiretu Robot (temporarily disabled for debugging) -->
+    <link name="blue_seiretu_base_link">
+        <inertial>
+            <origin rpy="0 0 0" xyz="1.8626252290206704 -0.5308186921199336 0.016889068327243004"/>
+            <mass value="2.198783634355126"/>
+            <inertia ixx="0.002972" ixy="-0.002307" ixz="0.004032" iyy="0.126512" iyz="0.000304" izz="0.127755"/>
+        </inertial>
+        <visual>
+            <origin rpy="0 0 0" xyz="0 0 0"/>
+            <geometry>
+                <mesh filename="package://blue_seiretu_description/meshes/base_link.stl" scale="0.001 0.001 0.001"/>
+            </geometry>
+            <material name="blue_seiretu_steel_satin"/>
+        </visual>
+        <collision>
+            <origin rpy="0 0 0" xyz="0 0 0"/>
+            <geometry>
+                <mesh filename="package://blue_seiretu_description/meshes/base_link.stl" scale="0.001 0.001 0.001"/>
+            </geometry>
+        </collision>
+    </link>
+    <link name="blue_seiretu_1">
+        <inertial>
+            <origin rpy="0 0 0" xyz="0.06569597903167557 -0.1195516608327013 0.09204470816379795"/>
+            <mass value="0.22394819815220426"/>
+            <inertia ixx="0.000651" ixy="-1.4e-05" ixz="-3.1e-05" iyy="0.000188" iyz="3.8e-05" izz="0.000754"/>
+        </inertial>
+        <visual>
+            <origin rpy="0 0 0" xyz="0.023506 0.51118 -0.019391"/>
+            <geometry>
+                <mesh filename="package://blue_seiretu_description/meshes/blue_seiretu_1.stl" scale="0.001 0.001 0.001"/>
+            </geometry>
+            <material name="blue_seiretu_steel_satin"/>
+        </visual>
+        <collision>
+            <origin rpy="0 0 0" xyz="0.023506 0.51118 -0.019391"/>
+            <geometry>
+                <mesh filename="package://blue_seiretu_description/meshes/blue_seiretu_1.stl" scale="0.001 0.001 0.001"/>
+            </geometry>
+        </collision>
+    </link>
+    <joint name="world_to_blue_seiretu" type="fixed">
+        <origin rpy="0 0 0" xyz="0.0 0.0 0.0"/>
+        <parent link="world"/>
+        <child link="blue_seiretu_base_link"/>
+    </joint>
+    <joint name="blue_slider" type="prismatic">
+        <origin rpy="0 0 0" xyz="-0.023506 -0.51118 0.019391"/>
+        <parent link="blue_seiretu_base_link"/>
+        <child link="blue_seiretu_1"/>
+        <axis xyz="1.0 -0.0 0.0"/>
+        <limit effort="100" lower="-0.457" upper="0.0" velocity="100"/>
+    </joint>
+    <!-- Red Seiretu Robot -->
+    <link name="red_seiretu_base_link">
+        <inertial>
+            <origin rpy="0 0 0" xyz="1.8626252290206704 -0.5308186921199336 0.016889068327243004"/>
+            <mass value="2.198783634355126"/>
+            <inertia ixx="0.002972" ixy="-0.002307" ixz="0.004032" iyy="0.126512" iyz="0.000304" izz="0.127755"/>
+        </inertial>
+        <visual>
+            <origin rpy="0 0 0" xyz="0 0 0"/>
+            <geometry>
+                <mesh filename="package://red_seiretu_description/meshes/base_link.stl" scale="0.001 0.001 0.001"/>
+            </geometry>
+            <material name="red_seiretu_steel_satin"/>
+        </visual>
+        <collision>
+            <origin rpy="0 0 0" xyz="0 0 0"/>
+            <geometry>
+                <mesh filename="package://red_seiretu_description/meshes/base_link.stl" scale="0.001 0.001 0.001"/>
+            </geometry>
+        </collision>
+    </link>
+    <link name="red_seiretu_2">
+        <inertial>
+            <origin rpy="0 0 0" xyz="0.06569597903167557 -0.1195516608327013 0.09204470816379795"/>
+            <mass value="0.22394819815220426"/>
+            <inertia ixx="0.000651" ixy="-1.4e-05" ixz="-3.1e-05" iyy="0.000188" iyz="3.8e-05" izz="0.000754"/>
+        </inertial>
+        <visual>
+            <origin rpy="0 0 0" xyz="0.023506 0.51118 -0.019391"/>
+            <geometry>
+                <mesh filename="package://red_seiretu_description/meshes/red_seiretu_2.stl" scale="0.001 0.001 0.001"/>
+            </geometry>
+            <material name="red_seiretu_steel_satin"/>
+        </visual>
+        <collision>
+            <origin rpy="0 0 0" xyz="0.023506 0.51118 -0.019391"/>
+            <geometry>
+                <mesh filename="package://red_seiretu_description/meshes/red_seiretu_2.stl" scale="0.001 0.001 0.001"/>
+            </geometry>
+        </collision>
+    </link>
+    <transmission name="blue_slider_tran">
+        <type>transmission_interface/SimpleTransmission</type>
+        <joint name="blue_slider">
+            <hardwareInterface>hardware_interface/EffortJointInterface</hardwareInterface>
+        </joint>
+        <actuator name="blue_slider_actr">
+            <hardwareInterface>hardware_interface/EffortJointInterface</hardwareInterface>
+            <mechanicalReduction>1</mechanicalReduction>
+        </actuator>
+    </transmission>
+    <transmission name="red_slider_tran">
+    <type>transmission_interface/SimpleTransmission</type>
+    <joint name="red_slider">
+        <hardwareInterface>hardware_interface/EffortJointInterface</hardwareInterface>
+    </joint>
+    <actuator name="red_slider_actr">
+        <hardwareInterface>hardware_interface/EffortJointInterface</hardwareInterface>
+        <mechanicalReduction>1</mechanicalReduction>
+    </actuator>
+    </transmission>
+    <joint name="world_to_red_seiretu" type="fixed">
+        <origin rpy="0 0 0" xyz="0.0 0.0 0.0"/>
+        <parent link="world"/>
+        <child link="red_seiretu_base_link"/>
+    </joint>
+    <joint name="red_slider" type="prismatic">
+        <origin rpy="0 0 0" xyz="-0.023506 -0.51118 0.019391"/>
+        <parent link="red_seiretu_base_link"/>
+        <child link="red_seiretu_2"/>
+        <axis xyz="1.0 -0.0 0.0"/>
+        <limit effort="100" lower="-0.457" upper="0.0" velocity="100"/>
+    </joint>
+    <ros2_control name="seiretu_robot" type="system">
+        <hardware>
+            <plugin>mock_components/GenericSystem</plugin>
+        </hardware>
+        <joint name="blue_slider">
+            <command_interface name="position"/>
+            <state_interface name="position"/>
+            <state_interface name="velocity"/>
+        </joint>
+        <joint name="red_slider">
+            <command_interface name="position"/>
+            <state_interface name="position"/>
+            <state_interface name="velocity"/>
+        </joint>
+    </ros2_control>
 </robot>

Commit message: 整列機のurdfの初期位置を修正

File: install/robot_config/share/robot_config/config/dual_arm.urdf.xacro (robot description, xacro)
@@ -526,17 +526,17 @@
     <link name="blue_seiretu_base_link">
         <inertial>
-            <origin rpy="0 0 0" xyz="1.8626252290206704 -0.5308186921199336 0.016889068327243004"/>
+            <origin xyz="1.8626252290206704 -0.5308186921199336 0.016889068327242983" rpy="0 0 0"/>
             <mass value="2.198783634355126"/>
-            <inertia ixx="0.002972" ixy="-0.002307" ixz="0.004032" iyy="0.126512" iyz="0.000304" izz="0.127755"/>
+            <inertia ixx="0.002972" iyy="0.126512" izz="0.127755" ixy="-0.002307" iyz="0.000304" ixz="0.004032"/>
         </inertial>
         <visual>
-            <origin rpy="0 0 0" xyz="0 0 0"/>
+            <origin xyz="0 0 0" rpy="0 0 0"/>
             <geometry>
                 <mesh filename="package://blue_seiretu_description/meshes/base_link.stl" scale="0.001 0.001 0.001"/>
             </geometry>
-            <material name="blue_seiretu_steel_satin"/>
+            <material name="steel_satin"/>
         </visual>
         <collision>
-            <origin rpy="0 0 0" xyz="0 0 0"/>
+            <origin xyz="0 0 0" rpy="0 0 0"/>
             <geometry>
                 <mesh filename="package://blue_seiretu_description/meshes/base_link.stl" scale="0.001 0.001 0.001"/>
@@ -546,17 +546,17 @@
     <link name="blue_seiretu_1">
         <inertial>
-            <origin rpy="0 0 0" xyz="0.06569597903167557 -0.1195516608327013 0.09204470816379795"/>
+            <origin xyz="0.12169597903167509 -0.11955166083269919 0.09204470816379676" rpy="0 0 0"/>
             <mass value="0.22394819815220426"/>
-            <inertia ixx="0.000651" ixy="-1.4e-05" ixz="-3.1e-05" iyy="0.000188" iyz="3.8e-05" izz="0.000754"/>
+            <inertia ixx="0.000651" iyy="0.000188" izz="0.000754" ixy="-1.4e-05" iyz="3.8e-05" ixz="-3.1e-05"/>
         </inertial>
         <visual>
-            <origin rpy="0 0 0" xyz="0.023506 0.51118 -0.019391"/>
+            <origin xyz="0.343506 0.51118 -0.019391" rpy="0 0 0"/>
             <geometry>
                 <mesh filename="package://blue_seiretu_description/meshes/blue_seiretu_1.stl" scale="0.001 0.001 0.001"/>
             </geometry>
-            <material name="blue_seiretu_steel_satin"/>
+            <material name="steel_satin"/>
         </visual>
         <collision>
-            <origin rpy="0 0 0" xyz="0.023506 0.51118 -0.019391"/>
+            <origin xyz="0.343506 0.51118 -0.019391" rpy="0 0 0"/>
             <geometry>
                 <mesh filename="package://blue_seiretu_description/meshes/blue_seiretu_1.stl" scale="0.001 0.001 0.001"/>
@@ -570,26 +570,26 @@
     </joint>
     <joint name="blue_slider" type="prismatic">
-        <origin rpy="0 0 0" xyz="-0.023506 -0.51118 0.019391"/>
+        <origin xyz="-0.343506 -0.51118 0.019391" rpy="0 0 0"/>
         <parent link="blue_seiretu_base_link"/>
         <child link="blue_seiretu_1"/>
         <axis xyz="1.0 -0.0 0.0"/>
-        <limit effort="100" lower="-0.457" upper="0.0" velocity="100"/>
+        <limit upper="0.193" lower="-0.193" effort="100" velocity="100"/>
     </joint>
     <!-- Red Seiretu Robot -->
     <link name="red_seiretu_base_link">
         <inertial>
-            <origin rpy="0 0 0" xyz="1.8626252290206704 -0.5308186921199336 0.016889068327243004"/>
+            <origin xyz="1.8626252290206704 -0.5308186921199336 0.016889068327242983" rpy="0 0 0"/>
             <mass value="2.198783634355126"/>
-            <inertia ixx="0.002972" ixy="-0.002307" ixz="0.004032" iyy="0.126512" iyz="0.000304" izz="0.127755"/>
+            <inertia ixx="0.002972" iyy="0.126512" izz="0.127755" ixy="-0.002307" iyz="0.000304" ixz="0.004032"/>
         </inertial>
         <visual>
-            <origin rpy="0 0 0" xyz="0 0 0"/>
+            <origin xyz="0 0 0" rpy="0 0 0"/>
             <geometry>
                 <mesh filename="package://red_seiretu_description/meshes/base_link.stl" scale="0.001 0.001 0.001"/>
             </geometry>
-            <material name="red_seiretu_steel_satin"/>
+            <material name="steel_satin"/>
         </visual>
         <collision>
-            <origin rpy="0 0 0" xyz="0 0 0"/>
+            <origin xyz="0 0 0" rpy="0 0 0"/>
             <geometry>
                 <mesh filename="package://red_seiretu_description/meshes/base_link.stl" scale="0.001 0.001 0.001"/>
@@ -599,17 +599,17 @@
     <link name="red_seiretu_2">
         <inertial>
-            <origin rpy="0 0 0" xyz="0.06569597903167557 -0.1195516608327013 0.09204470816379795"/>
+            <origin xyz="0.12169597903168072 -0.11955166083270086 0.09204470816379565" rpy="0 0 0"/>
             <mass value="0.22394819815220426"/>
-            <inertia ixx="0.000651" ixy="-1.4e-05" ixz="-3.1e-05" iyy="0.000188" iyz="3.8e-05" izz="0.000754"/>
+            <inertia ixx="0.000651" iyy="0.000188" izz="0.000754" ixy="-1.4e-05" iyz="3.8e-05" ixz="-3.1e-05"/>
         </inertial>
         <visual>
-            <origin rpy="0 0 0" xyz="0.023506 0.51118 -0.019391"/>
+            <origin xyz="-1.916494 0.51118 -0.019391" rpy="0 0 0"/>
             <geometry>
                 <mesh filename="package://red_seiretu_description/meshes/red_seiretu_2.stl" scale="0.001 0.001 0.001"/>
             </geometry>
-            <material name="red_seiretu_steel_satin"/>
+            <material name="steel_satin"/>
         </visual>
         <collision>
-            <origin rpy="0 0 0" xyz="0.023506 0.51118 -0.019391"/>
+            <origin xyz="-1.916494 0.51118 -0.019391" rpy="0 0 0"/>
             <geometry>
                 <mesh filename="package://red_seiretu_description/meshes/red_seiretu_2.stl" scale="0.001 0.001 0.001"/>
@@ -643,9 +643,9 @@
     </joint>
     <joint name="red_slider" type="prismatic">
-        <origin rpy="0 0 0" xyz="-0.023506 -0.51118 0.019391"/>
+        <origin xyz="1.916494 -0.51118 0.019391" rpy="0 0 0"/>
         <parent link="red_seiretu_base_link"/>
         <child link="red_seiretu_2"/>
-        <axis xyz="1.0 -0.0 0.0"/>
-        <limit effort="100" lower="-0.457" upper="0.0" velocity="100"/>
+        <axis xyz="1.0 0.0 -0.0"/>
+        <limit upper="0.193" lower="-0.193" effort="100" velocity="100"/>
     </joint>
     <ros2_control name="seiretu_robot" type="system">

Commit message: ittannhozonn

File: install/robot_config/share/robot_config/config/dual_arm.urdf.xacro (robot description, xacro)
@@ -278,5 +278,5 @@
         </link>
         <!-- Joints for this arm instance -->
-        <joint name="${prefix}Revolute_1" type="continuous">
+        <joint name="${prefix}Revolute_1" type="revolute">
             <origin rpy="${Revolute_1_rpy}" xyz="${Revolute_1_xyz}"/>
             <parent link="${prefix}base_link"/>
